Commit message: Add dual FMCW radar tracking and aiming

File: catkin_ws/src/aiming_robot/urdf/shooter.urdf (robot description, URDF)
Before this commit: robot shooter, 3 links, 2 joints
Links:
- added link radar_left_link
- added link radar_right_link
Joints:
- added joint radar_left_mount: type fixed, parent base_link, child radar_left_link, origin xyz=0 0.14 1.45 rpy=0 0 0
- added joint radar_right_mount: type fixed, parent base_link, child radar_right_link, origin xyz=0 -0.14 1.45 rpy=0 0 0

Commit message: Add visible camera and radar sensor housings

File: catkin_ws/src/aiming_robot/urdf/shooter.urdf (robot description, URDF)
Before this commit: robot shooter, 5 links, 4 joints
Links:
- link radar_left_link: geometry visual box size=0.015 0.17 0.11; visual box size=0.075 0.022 0.022
- link radar_right_link: geometry visual box size=0.015 0.17 0.11; visual box size=0.075 0.022 0.022
- link tilt_link: geometry collision cylinder length=0.3 radius=0.04; visual box size=0.22 0.17 0.14

Commit message: Improve single-radar tracking and display

File: catkin_ws/src/aiming_robot/urdf/shooter.urdf (robot description, URDF)
Before this commit: robot shooter, 5 links, 4 joints
Links:
- removed link radar_right_link
- link radar_left_link: geometry visual box size=0.015 0.17 0.11; visual box size=0.075 0.022 0.022
Joints:
- removed joint radar_right_mount
- joint radar_left_mount: origin xyz=0 0.14 1.45 rpy=0 0 0 -> xyz=0 1.50 1.45 rpy=0 0 0
